Commit message: temp

File: urdf/saber_750d.urdf (robot description, URDF)
Before this commit: robot hex_ros_ik_saber_750d, 7 links, 6 joints
Links:
- added link link_7, mass 0.0295686940024556; collision mesh filename=package://xpkg_urdf_saber/meshes/link_7.STL; visual mesh filename=package://xpkg_urdf_saber/meshes/link_7.STL
- link base_link: mass 1.075 -> 0.556279812163046; geometry collision mesh filename=package://xpkg_urdf_saber/meshes/base_link.STL; visual mesh filename=package://xpkg_urdf_saber/meshes/base_link.STL
- link link_1: mass 1.04678 -> 0.210052072515294; geometry collision mesh filename=package://xpkg_urdf_saber/meshes/link_1.STL; visual mesh filename=package://xpkg_urdf_saber/meshes/link_1.STL
- link link_2: mass 1.366628 -> 0.546006723511329; geometry collision mesh filename=package://xpkg_urdf_saber/meshes/link_2.STL; visual mesh filename=package://xpkg_urdf_saber/meshes/link_2.STL
- link link_3: mass 0.802284 -> 0.507512757354665; geometry collision mesh filename=package://xpkg_urdf_saber/meshes/link_3.STL; visual mesh filename=package://xpkg_urdf_saber/meshes/link_3.STL
- link link_4: mass 0.907814 -> 0.462861602611646; geometry collision mesh filename=package://xpkg_urdf_saber/meshes/link_4.STL; visual mesh filename=package://xpkg_urdf_saber/meshes/link_4.STL
- link link_5: mass 0.66461 -> 0.726565505856402; geometry collision mesh filename=package://xpkg_urdf_saber/meshes/link_5.STL; visual mesh filename=package://xpkg_urdf_saber/meshes/link_5.STL
- link link_6: mass 0.0 -> 0.281670524443241; geometry collision mesh filename=package://xpkg_urdf_saber/meshes/link_6.STL; visual mesh filename=package://xpkg_urdf_saber/meshes/link_6.STL
Joints:
- added joint joint_7: type revolute, parent link_6, child link_7, origin xyz=0.095 0 0 rpy=1.5708 0 1.5708, axis 0 0 1, limit lower=-3.14 upper=3.14 effort=0 velocity=0
- joint joint_1: limit lower=-2.9670597283903604 upper=2.9670597283903604 effort=40.0 velocity=1.0 -> lower=-2.07 upper=2.07 effort=0 velocity=0; origin xyz=0.0075 0 0.0895 rpy=1.5707963268 -1.5707963268 3.14159265359 -> xyz=0.008 0 0.085 rpy=1.5708 -1.5708 0
- joint joint_2: axis 0 0 1 -> 0 0 -1; limit lower=-1.5707963268 upper=1.5707963268 effort=40.0 velocity=1.0 -> lower=-1.57 upper=1.57 effort=0 velocity=0; origin xyz=0.043 0 0 rpy=0 0 -1.5707963268 -> xyz=0.048 0 0 rpy=0 0 -1.5708
- joint joint_3: axis 0 0 -1 -> 1 0 0; limit lower=-1.0471975512 upper=3.14159265359 effort=40.0 velocity=1.0 -> lower=-2.79 upper=2.79 effort=0 velocity=0; origin xyz=0 0.3268 0 rpy=3.14159265359 0 1.5707963268 -> xyz=0 0.121 0 rpy=-0.14087 0.0047123 1.604
- joint joint_4: axis 1 0 0 -> 0 0 1; limit lower=-2.79252680319 upper=2.79252680319 effort=40.0 velocity=1.0 -> lower=-1.57 upper=1.57 effort=0 velocity=0; origin xyz=0.08847 0.072 -7.0034E-05 rpy=1.5707963268 0 0 -> xyz=0.13642 -0.0045787 0 rpy=-3.0006 0 -0.03355
- joint joint_5: axis 0 0 1 -> 1 0 0; limit lower=-1.5707963268 upper=1.5707963268 effort=40.0 velocity=1.0 -> lower=-2.79 upper=2.79 effort=0 velocity=0; origin xyz=0.206 0 0 rpy=1.5707963268 0 0 -> xyz=0.1325 0 0 rpy=1.5708 0 0
- joint joint_6: axis 0 0 1 -> 0 0 -1; limit lower=-2.9670597283903604 upper=2.9670597283903604 effort=40.0 velocity=1.0 -> lower=-1.57 upper=1.57 effort=0 velocity=0; origin xyz=0.11 0 0 rpy=1.5707963268 0.0 1.5707963268 -> xyz=0.17204 0 0 rpy=1.5708 0 0

Commit message: temp

File: urdf/saber_750d.urdf (robot description, URDF)
Before this commit: robot xpkg_urdf_saber, 8 links, 7 joints
Links:
- link base_link: geometry collision mesh filename=package://hex_ros_ik_saber_750d/urdf/meshes/base_link.STL; visual mesh filename=package://hex_ros_ik_saber_750d/urdf/meshes/base_link.STL
- link link_1: geometry collision mesh filename=package://hex_ros_ik_saber_750d/urdf/meshes/link_1.STL; visual mesh filename=package://hex_ros_ik_saber_750d/urdf/meshes/link_1.STL
- link link_2: geometry collision mesh filename=package://hex_ros_ik_saber_750d/urdf/meshes/link_2.STL; visual mesh filename=package://hex_ros_ik_saber_750d/urdf/meshes/link_2.STL
- link link_3: geometry collision mesh filename=package://hex_ros_ik_saber_750d/urdf/meshes/link_3.STL; visual mesh filename=package://hex_ros_ik_saber_750d/urdf/meshes/link_3.STL
- link link_4: geometry collision mesh filename=package://hex_ros_ik_saber_750d/urdf/meshes/link_4.STL; visual mesh filename=package://hex_ros_ik_saber_750d/urdf/meshes/link_4.STL
- link link_5: geometry collision mesh filename=package://hex_ros_ik_saber_750d/urdf/meshes/link_5.STL; visual mesh filename=package://hex_ros_ik_saber_750d/urdf/meshes/link_5.STL
- link link_6: geometry collision mesh filename=package://hex_ros_ik_saber_750d/urdf/meshes/link_6.STL; visual mesh filename=package://hex_ros_ik_saber_750d/urdf/meshes/link_6.STL
- link link_7: geometry collision mesh filename=package://hex_ros_ik_saber_750d/urdf/meshes/link_7.STL; visual mesh filename=package://hex_ros_ik_saber_750d/urdf/meshes/link_7.STL

Commit message: temp

File: urdf/saber_750d.urdf (robot description, URDF)
Before this commit: robot xpkg_urdf_saber, 8 links, 7 joints
Joints:
- joint joint_7: origin xyz=0.095 0 0 rpy=1.5708 0 1.5708 -> xyz=0.095 0 0 rpy=-1.5708 0 -1.5708
